File: Reproduction_PCBs/Main_PCB/opticalblock.kicad_sch (KiCad schematic)
At the start: 34 parts, among them CN102 FFC_Conn_01x12, IC101 CXA1081M, P103 Conn_01x06_Pin, Q101 2SB1132

Commit message: Final commit before ordering
Parts:
- removed C102: 3.3uF, Capacitor_SMD:CP_Elec_4x5.4, symbol Device:C_Polarized
- added C102: 3.3uF, Capacitor_SMD:C_0805_2012Metric, symbol Device:C
Connections:
- net VC: now also C102.2
- net at CN102.7 (Pin_7), R102.1: now also C102.1
Changed lines of the file:
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@@
 	(title_block
 		(title "PC-Engine CDR-30A (CD-ROM2) MAIN PWR Reproduction")
-		(date "2025-02-24")
+		(date "2025-02-26")
 		(rev "0.1")
 		(company "Author: Regis Galland")
@@
 	)
 	(symbol
-		(lib_id "Device:C_Polarized")
-		(at 95.25 116.84 0)
-		(unit 1)
-		(exclude_from_sim no)
-		(in_bom yes)
-		(on_board yes)
-		(dnp no)
-		(fields_autoplaced yes)
-		(property "Reference" "C102"
-			(at 98.171 114.7388 0)
-			(effects
-				(font
-					(size 1.27 1.27)
-				)
-				(justify left)
-			)
-		)
-		(property "Value" "3.3uF"
-			(at 98.171 117.1631 0)
-			(effects
-				(font
-					(size 1.27 1.27)
-				)
-				(justify left)
-			)
-		)
-		(property "Footprint" "Capacitor_SMD:CP_Elec_4x5.4"
-			(at 96.2152 120.65 0)
-			(effects
-				(font
-					(size 1.27 1.27)
-				)
-				(hide yes)
-			)
-		)
-		(property "Datasheet" "~"
-			(at 95.25 116.84 0)
-			(effects
-				(font
-					(size 1.27 1.27)
-				)
-				(hide yes)
-			)
-		)
-		(property "Description" ""
-			(at 95.25 116.84 0)
-			(effects
-				(font
-					(size 1.27 1.27)
-				)
-				(hide yes)
-			)
-		)
-		(pin "1"
-		)
-		(pin "2"
-		)
-		(instances
-			(project "MAIN_PWR"
-				(path "/035ab33a-1caf-4155-b57e-664ce0b37194/56cfd0d5-32ce-4b42-8ead-ceb694bb000b"
-					(reference "C102")
-					(unit 1)
-				)
-			)
-		)
-	)
-	(symbol
 		(lib_id "power:GND")
 		(at 233.68 93.98 0)
@@
 					(unit 1)
 				)
+			)
+		)
+	)
+	(symbol
+		(lib_id "Device:C")
+		(at 95.25 116.84 0)
+		(unit 1)
+		(exclude_from_sim no)
+		(in_bom yes)
+		(on_board yes)
+		(dnp no)
+		(property "Reference" "C102"
+			(at 90.17 118.364 0)
+			(effects
+				(font
+					(size 1.27 1.27)
+				)
+			)
+		)
+		(property "Value" "3.3uF"
+			(at 89.662 115.57 0)
+			(effects
+				(font
+					(size 1.27 1.27)
+				)
+			)
+		)
+		(property "Footprint" "Capacitor_SMD:C_0805_2012Metric"
+			(at 96.2152 120.65 0)
+			(effects
+				(font
+					(size 1.27 1.27)
+				)
+				(hide yes)
+			)
+		)
+		(property "Datasheet" "~"
+			(at 95.25 116.84 0)
+			(effects
+				(font
+					(size 1.27 1.27)
+				)
+				(hide yes)
+			)
+		)
+		(property "Description" ""
+			(at 95.25 116.84 0)
+			(effects
+				(font
+					(size 1.27 1.27)
+				)
+				(hide yes)
+			)
+		)
+		(pin "1"
+		)
+		(pin "2"
+		)
+		(instances
+			(project "Main_PCB"
+				(path "/035ab33a-1caf-4155-b57e-664ce0b37194/56cfd0d5-32ce-4b42-8ead-ceb694bb000b"
+					(reference "C102")
+					(unit 1)
+				)
