File: Reproduction_PCBs/Main_PCB/scsi.kicad_sch (KiCad schematic)
At the start: 66 parts, among them IC107 D4364G, IC109 D6378GF, IC301 L7805, IC302 1951A, Q104 2SC2412K

Commit message: Final commit before ordering
Parts:
- removed R534: 0, Resistor_SMD:R_0603_1608Metric, symbol Device:R
- IC107: footprint Package_SO:SOIC-28W_7.5x17.9mm_P1.27mm -> Package_SO:SOP-28_8.4x18.16mm_P1.27mm
Connections:
- net at IC109.90 (XIN): now also C150.2, C151.1, Q104.2 (E), R167.2
Other:
- note removed: "No R534 on CDR-30 Rev"
Changed lines of the file:
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@@
 	(title_block
 		(title "PC-Engine CDR-30A (CD-ROM2) MAIN PWR Reproduction")
-		(date "2025-02-24")
+		(date "2025-02-26")
 		(rev "0.1")
 		(company "Author: Regis Galland")
@@
 	(wire
 		(pts
-			(xy 29.21 149.86) (xy 36.83 149.86)
+			(xy 29.21 149.86) (xy 57.15 149.86)
 		)
 		(stroke
@@
 	(wire
 		(pts
-			(xy 44.45 149.86) (xy 57.15 149.86)
-		)
-		(stroke
-			(width 0)
-			(type default)
-		)
-	)
-	(wire
-		(pts
 			(xy 292.1 104.14) (xy 314.96 104.14)
 		)
@@
 		)
 	)
-	(text "No R534 on CDR-30 Rev"
-		(exclude_from_sim no)
-		(at 36.068 146.304 0)
-		(effects
-			(font
-				(size 1.27 1.27)
-			)
-		)
-	)
 	(text "30-way IFU facing connector"
 		(exclude_from_sim no)
@@
 	(symbol
 		(lib_id "Device:R")
-		(at 40.64 149.86 270)
-		(mirror x)
-		(unit 1)
-		(exclude_from_sim no)
-		(in_bom yes)
-		(on_board yes)
-		(dnp no)
-		(property "Reference" "R534"
-			(at 49.276 148.59 90)
-			(effects
-				(font
-					(size 1.27 1.27)
-				)
-				(justify right)
-			)
-		)
-		(property "Value" "0"
-			(at 41.402 149.86 90)
-			(effects
-				(font
-					(size 1.27 1.27)
-				)
-				(justify right)
-			)
-		)
-		(property "Footprint" "Resistor_SMD:R_0603_1608Metric"
-			(at 40.64 151.638 90)
-			(effects
-				(font
-					(size 1.27 1.27)
-				)
-				(hide yes)
-			)
-		)
-		(property "Datasheet" "~"
-			(at 40.64 149.86 0)
-			(effects
-				(font
-					(size 1.27 1.27)
-				)
-				(hide yes)
-			)
-		)
-		(property "Description" ""
-			(at 40.64 149.86 0)
-			(effects
-				(font
-					(size 1.27 1.27)
-				)
-				(hide yes)
-			)
-		)
-		(pin "1"
-		)
-		(pin "2"
-		)
-		(instances
-			(project "MAIN_PWR"
-				(path "/035ab33a-1caf-4155-b57e-664ce0b37194/c7b0ff97-3379-4f62-addb-1558cc68b0b5"
-					(reference "R534")
-					(unit 1)
-				)
-			)
-		)
-	)
-	(symbol
-		(lib_id "Device:R")
 		(at 367.03 104.14 270)
 		(mirror x)
@@
 			)
 		)
-		(property "Footprint" "Package_SO:SOIC-28W_7.5x17.9mm_P1.27mm"
+		(property "Footprint" "Package_SO:SOP-28_8.4x18.16mm_P1.27mm"
 			(at 223.52 46.99 0)
 			(effects
